File: kicad/ckt-signal/ckt-signal.kicad_pcb (KiCad board)
At the start: 2 copper layers, 12.7 x 60.3 mm, 8 parts, among them J1 Screw_Terminal_01x04

Commit message: Add version text to single head signal
Other:
- board text added: "CKT-SIGNAL v3.0"
- board text added: "Iowa Scaled Engineering"
- board text added: "iascaled.com"
Changed lines of the file:
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@@
   (gr_line (start 26.035 190.246) (end 38.735 190.246) (layer "Edge.Cuts") (width 0.1))
   (gr_arc (start 35.814 138.43) (mid 35.337012 140.19434) (end 34.036 141.478) (layer "Edge.Cuts") (width 0.1))
+  (gr_text "CKT-SIGNAL\nv3.0" (at 32.385 178.181) (layer "B.SilkS")
+    (effects (font (size 1 1) (thickness 0.15)) (justify mirror))
+  )
+  (gr_text "Iowa Scaled\nEngineering" (at 32.385 174.752) (layer "B.SilkS")
+    (effects (font (size 1 1) (thickness 0.15)) (justify mirror))
+  )
+  (gr_text "iascaled.com" (at 32.385 188.595) (layer "B.SilkS")
+    (effects (font (size 1 1) (thickness 0.15)) (justify mirror))
+  )
   (gr_text "+" (at 36.195 188.722) (layer "F.SilkS")
     (effects (font (size 1.524 1.524) (thickness 0.15)))
