File: kicad/ckt-signal/ckt-signal-array.kicad_pcb (KiCad board)
At the start: 2 copper layers, 75.6 x 165.1 mm, 166 parts, among them J1 Screw_Terminal_01x04

Commit message: Repanelize the 1x signals
Parts:
- removed the D1 at (170.2, 79.7)
- removed the R3 at (130.9, 111.4)
- removed the REF** at (178.7, 22.5) (x2)
- removed the REF** at (118.3, 22.5) (x2)
- removed the REF** at (118.3, 182.6) (x2)
- added J1: Screw_Terminal_01x04, TerminalBlock_Phoenix:TerminalBlock_Phoenix_MPT-0,5-4-2.54_1x04_P2.54mm_Horizontal, F.Cu at (124.9, 106.4)
- added R2: 1k, Resistor_SMD:R_0805_2012Metric, F.Cu at (130.9, 78.4)
- added REF**: Fiducial, Fiducial, F.Cu at (118.3, 22.5)
- added REF**: Fiducial, Fiducial, F.Cu at (118.3, 182.6)
- added REF**: Fiducial, Fiducial, F.Cu at (178.7, 22.5)
- added REF**: Fiducial, Fiducial, B.Cu at (118.3, 182.6)
- added REF**: Fiducial, Fiducial, B.Cu at (118.3, 22.5)
- added REF**: Fiducial, Fiducial, B.Cu at (178.7, 22.5)
- D1: renamed from R2; value 1k -> RED; footprint Resistor_SMD:R_0805_2012Metric -> LED_SMD:LED_0805_2012Metric
- R3: renamed from J1; value Screw_Terminal_01x04 -> 1k; footprint TerminalBlock_Phoenix:TerminalBlock_Phoenix_MPT-0,5-4-2.54_1x04_P2.54mm_Horizontal -> Resistor_SMD:R_0805_2012Metric
- moved D1 39.3 mm to (170.2, 79.7), turned to -90 degrees
- moved R3 7.84 mm to (130.9, 111.4), turned to 180 degrees
Connections:
- D1 pad 1: Board_3-Net-(D2-Pad1) -> Board_3-Net-(D1-Pad1)
- D1 pad 2: Board_3-Net-(J1-Pad2) -> Board_3-Net-(D1-Pad2)
- R3 pad 1: Board_5-Net-(J1-Pad1) -> Board_5-Net-(D3-Pad1)
- R3 pad 2: Board_5-Net-(J1-Pad2) -> Board_5-Net-(J1-Pad3)
Other:
- board text added: "CKT-SIGNAL v3.0"
- board text added: "Iowa Scaled Engineering"
- board text added: "iascaled.com"
