File: kicad/ckt-signal-2x/ckt-signal-2x.kicad_pcb (KiCad board)
At the start: 2 copper layers, 22.9 x 66.7 mm, 14 parts, among them J1 Screw_Terminal_01x08

Commit message: Fixed Nathan's dangling traces
Changed lines of the file:
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@@
       (effects (font (size 0.5 0.5) (thickness 0.08)))
     )
+    (fp_line (start -1.685 -0.96) (end -1.685 0.96) (layer "F.SilkS") (width 0.12))
     (fp_line (start -1.685 0.96) (end 1 0.96) (layer "F.SilkS") (width 0.12))
-    (fp_line (start -1.685 -0.96) (end -1.685 0.96) (layer "F.SilkS") (width 0.12))
     (fp_line (start 1 -0.96) (end -1.685 -0.96) (layer "F.SilkS") (width 0.12))
     (fp_line (start -1.68 0.95) (end -1.68 -0.95) (layer "F.CrtYd") (width 0.05))
     (fp_line (start -1.68 -0.95) (end 1.68 -0.95) (layer "F.CrtYd") (width 0.05))
-    (fp_line (start 1.68 -0.95) (end 1.68 0.95) (layer "F.CrtYd") (width 0.05))
-    (fp_line (start 1.68 0.95) (end -1.68 0.95) (layer "F.CrtYd") (width 0.05))
+    (fp_line (start 1.68 0.95) (end -1.68 0.95) (layer "F.CrtYd") (width 0.05))
+    (fp_line (start 1.68 -0.95) (end 1.68 0.95) (layer "F.CrtYd") (width 0.05))
+    (fp_line (start 1 -0.6) (end -0.7 -0.6) (layer "F.Fab") (width 0.1))
+    (fp_line (start -0.7 -0.6) (end -1 -0.3) (layer "F.Fab") (width 0.1))
+    (fp_line (start -1 -0.3) (end -1 0.6) (layer "F.Fab") (width 0.1))
     (fp_line (start -1 0.6) (end 1 0.6) (layer "F.Fab") (width 0.1))
     (fp_line (start 1 0.6) (end 1 -0.6) (layer "F.Fab") (width 0.1))
-    (fp_line (start -1 -0.3) (end -1 0.6) (layer "F.Fab") (width 0.1))
-    (fp_line (start 1 -0.6) (end -0.7 -0.6) (layer "F.Fab") (width 0.1))
-    (fp_line (start -0.7 -0.6) (end -1 -0.3) (layer "F.Fab") (width 0.1))
     (pad "1" smd roundrect (at -0.9375 0) (size 0.975 1.4) (layers "F.Cu" "F.Paste" "F.Mask") (roundrect_rratio 0.25)
       (net 6 "Net-(D5-Pad1)") (pinfunction "K") (pintype "passive"))
@@
     )
     (fp_line (start 1 -0.96) (end -1.685 -0.96) (layer "F.SilkS") (width 0.12))
+    (fp_line (start -1.685 -0.96) (end -1.685 0.96) (layer "F.SilkS") (width 0.12))
     (fp_line (start -1.685 0.96) (end 1 0.96) (layer "F.SilkS") (width 0.12))
-    (fp_line (start -1.685 -0.96) (end -1.685 0.96) (layer "F.SilkS") (width 0.12))
-    (fp_line (start -1.68 0.95) (end -1.68 -0.95) (layer "F.CrtYd") (width 0.05))
-    (fp_line (start 1.68 -0.95) (end 1.68 0.95) (layer "F.CrtYd") (width 0.05))
-    (fp_line (start -1.68 -0.95) (end 1.68 -0.95) (layer "F.CrtYd") (width 0.05))
-    (fp_line (start 1.68 0.95) (end -1.68 0.95) (layer "F.CrtYd") (width 0.05))
+    (fp_line (start 1.68 0.95) (end -1.68 0.95) (layer "F.CrtYd") (width 0.05))
+    (fp_line (start -1.68 0.95) (end -1.68 -0.95) (layer "F.CrtYd") (width 0.05))
+    (fp_line (start -1.68 -0.95) (end 1.68 -0.95) (layer "F.CrtYd") (width 0.05))
+    (fp_line (start 1.68 -0.95) (end 1.68 0.95) (layer "F.CrtYd") (width 0.05))
     (fp_line (start 1 0.6) (end 1 -0.6) (layer "F.Fab") (width 0.1))
-    (fp_line (start -1 -0.3) (end -1 0.6) (layer "F.Fab") (width 0.1))
-    (fp_line (start -1 0.6) (end 1 0.6) (layer "F.Fab") (width 0.1))
     (fp_line (start 1 -0.6) (end -0.7 -0.6) (layer "F.Fab") (width 0.1))
     (fp_line (start -0.7 -0.6) (end -1 -0.3) (layer "F.Fab") (width 0.1))
+    (fp_line (start -1 0.6) (end 1 0.6) (layer "F.Fab") (width 0.1))
+    (fp_line (start -1 -0.3) (end -1 0.6) (layer "F.Fab") (width 0.1))
     (pad "1" smd roundrect (at -0.9375 0) (size 0.975 1.4) (layers "F.Cu" "F.Paste" "F.Mask") (roundrect_rratio 0.25)
       (net 4 "Net-(D4-Pad1)") (pinfunction "K") (pintype "passive"))
@@
       (effects (font (size 0.5 0.5) (thickness 0.08)))
     )
+    (fp_line (start -1.685 0.96) (end 1 0.96) (layer "F.SilkS") (width 0.12))
     (fp_line (start -1.685 -0.96) (end -1.685 0.96) (layer "F.SilkS") (width 0.12))
     (fp_line (start 1 -0.96) (end -1.685 -0.96) (layer "F.SilkS") (width 0.12))
-    (fp_line (start -1.685 0.96) (end 1 0.96) (layer "F.SilkS") (width 0.12))
-    (fp_line (start -1.68 0.95) (end -1.68 -0.95) (layer "F.CrtYd") (width 0.05))
-    (fp_line (start 1.68 0.95) (end -1.68 0.95) (layer "F.CrtYd") (width 0.05))
-    (fp_line (start -1.68 -0.95) (end 1.68 -0.95) (layer "F.CrtYd") (width 0.05))
-    (fp_line (start 1.68 -0.95) (end 1.68 0.95) (layer "F.CrtYd") (width 0.05))
+    (fp_line (start -1.68 -0.95) (end 1.68 -0.95) (layer "F.CrtYd") (width 0.05))
+    (fp_line (start 1.68 -0.95) (end 1.68 0.95) (layer "F.CrtYd") (width 0.05))
+    (fp_line (start 1.68 0.95) (end -1.68 0.95) (layer "F.CrtYd") (width 0.05))
+    (fp_line (start -1.68 0.95) (end -1.68 -0.95) (layer "F.CrtYd") (width 0.05))
+    (fp_line (start -0.7 -0.6) (end -1 -0.3) (layer "F.Fab") (width 0.1))
+    (fp_line (start -1 0.6) (end 1 0.6) (layer "F.Fab") (width 0.1))
+    (fp_line (start -1 -0.3) (end -1 0.6) (layer "F.Fab") (width 0.1))
     (fp_line (start 1 -0.6) (end -0.7 -0.6) (layer "F.Fab") (width 0.1))
-    (fp_line (start -1 0.6) (end 1 0.6) (layer "F.Fab") (width 0.1))
-    (fp_line (start -0.7 -0.6) (end -1 -0.3) (layer "F.Fab") (width 0.1))
     (fp_line (start 1 0.6) (end 1 -0.6) (layer "F.Fab") (width 0.1))
-    (fp_line (start -1 -0.3) (end -1 0.6) (layer "F.Fab") (width 0.1))
     (pad "1" smd roundrect (at -0.9375 0) (size 0.975 1.4) (layers "F.Cu" "F.Paste" "F.Mask") (roundrect_rratio 0.25)
       (net 3 "Net-(D3-Pad1)") (pinfunction "K") (pintype "passive"))
@@
   (gr_line (start 30.734 149.987) (end 30.734 160.909) (layer "Edge.Cuts") (width 0.1))
   (gr_line (start 28.956 127) (end 28.956 132.08) (layer "Edge.Cuts") (width 0.1))
-  (gr_arc (start 30.734 149.987) (mid 29.432998 148.703337) (end 28.956 146.939) (layer "Edge.Cuts") (width 0.1))
+  (gr_arc (start 30.734 149.987) (mid 29.432997 148.703335) (end 28.956 146.939) (layer "Edge.Cuts") (width 0.1))
   (gr_arc (start 30.734 135.128) (mid 29.432997 133.844335) (end 28.956 132.08) (layer "Edge.Cuts") (width 0.1))
   (gr_line (start 28.956 141.859) (end 28.956 146.939) (layer "Edge.Cuts") (width 0.1))
@@
   (gr_line locked (start 20.955 190.246) (end 43.815 190.246) (layer "Edge.Cuts") (width 0.1))
   (gr_line (start 20.955 190.246) (end 20.955 172.466) (layer "Edge.Cuts") (width 0.1))
-  (gr_arc (start 35.814 146.939) (mid 35.337014 148.703344) (end 34.036 149.987) (layer "Edge.Cuts") (width 0.1))
+  (gr_arc (start 35.814 146.939) (mid 35.337015 148.703342) (end 34.036 149.987) (layer "Edge.Cuts") (width 0.1))
   (gr_line (start 34.036 135.128) (end 34.036 138.811) (layer "Edge.Cuts") (width 0.1))
   (gr_text "Iowa Scaled Engineering\nCKT-SIGNAL-2X v3.0\n©2024 www.iascaled.com" (at 32.258 177.927) (layer "B.SilkS")
@@
   (segment (start 36.576 166.243) (end 36.576 171.831) (width 0.254) (layer "F.Cu") (net 4))
   (segment (start 36.195 172.212) (end 36.195 176.7605) (width 0.254) (layer "F.Cu") (net 4))
-  (segment (start 31.75 132.3825) (end 31.4475 132.08) (width 0.254) (layer "F.Cu") (net 4))
   (segment (start 31.4475 133.1445) (end 30.988 133.604) (width 0.254) (layer "F.Cu") (net 4))
   (segment (start 34.671 164.338) (end 36.576 166.243) (width 0.254) (layer "F.Cu") (net 4))
@@
   (segment (start 23.495 178.5855) (end 23.495 184.023) (width 0.254) (layer "F.Cu") (net 9))
   (segment (start 26.035 184.023) (end 26.035 178.5855) (width 0.254) (layer "F.Cu") (net 10))
-  (segment (start 28.57 178.5905) (end 28.575 178.5855) (width 0.254) (layer "F.Cu") (net 11))
   (segment (start 28.575 184.023) (end 28.575 178.5855) (width 0.254) (layer "F.Cu") (net 11))
   (segment (start 36.195 178.5855) (end 36.195 184.023) (width 0.254) (layer "F.Cu") (net 12))
